File: GPS.kicad_sch (KiCad schematic)
At the start: 0 parts

Commit message: changes
Other:
- note added: "GPS"
- note added: "Implement GPS to be used as part of the rocket's state estimation solution. We should implement one that is rated for the g forces, is very common, and provides good accuracy. It should also have an external antenna, and we should route it through an SMA connector. the MAX-M10S-00B seems like a good option."
Changed lines of the file:
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@@
 	(generator_version "10.0")
 	(paper "A4")
+	(text "GPS"
+		(exclude_from_sim no)
+		(at 19.812 21.844 0)
+		(effects
+			(font
+				(size 2.54 2.54)
+				(thickness 0.508)
+				(bold yes)
+			)
+		)
+	)
+	(text "Implement GPS to be used as part of the rocket's state estimation solution.\nWe should implement one that is rated for the g forces, is very common, and provides good accuracy.\nIt should also have an external antenna, and we should route it through an SMA connector.\n\nthe MAX-M10S-00B seems like a good option."
+		(exclude_from_sim no)
+		(at 16.256 30.48 0)
+		(effects
+			(font
+				(size 1.27 1.27)
+			)
+			(justify left)
+		)
+	)
 )
