File: Radio.kicad_sch (KiCad schematic)
At the start: 0 parts

Commit message: changes
Other:
- note added: "Radio"
- note added: "The radio on this board has to interface with the one on the groundstation. Talk to Andrew about what he is using and make sure they agree. It is a LoRa transceiver of some sort, just make sure it is compatible with Andrew's design. Also add UART connector, JST-GH, if we ever want to connect to an external radio like the RFD 900x"
Changed lines of the file:
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@@
 	(generator_version "10.0")
 	(paper "A4")
+	(text "Radio"
+		(exclude_from_sim no)
+		(at 25.4 18.796 0)
+		(effects
+			(font
+				(size 2.54 2.54)
+				(thickness 0.508)
+				(bold yes)
+			)
+		)
+	)
+	(text "The radio on this board has to interface with the one on the groundstation.\nTalk to Andrew about what he is using and make sure they agree.\n\nIt is a LoRa transceiver of some sort, just make sure it is compatible with Andrew's design.\n\nAlso add UART connector, JST-GH, if we ever want to connect to an external radio like\nthe RFD 900x"
+		(exclude_from_sim no)
+		(at 20.32 29.718 0)
+		(effects
+			(font
+				(size 1.27 1.27)
+			)
+			(justify left)
+		)
+	)
 )
