File: MCU.kicad_sch (KiCad schematic)
At the start: 0 parts

Commit message: changes
Other:
- note added: "Implement the core processor of the flight computer. This is relatively simple, and the main complexity comes from determining which pins should be broken out."
- note added: "Microcontroller"
Changed lines of the file:
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@@
 	(generator "eeschema")
 	(generator_version "10.0")
-	(paper "A4")
+	(paper "A3")
+	(text "Implement the core processor of the flight computer.\nThis is relatively simple, and the main complexity comes from \ndetermining which pins should be broken out."
+		(exclude_from_sim no)
+		(at 18.542 28.956 0)
+		(effects
+			(font
+				(size 1.27 1.27)
+			)
+			(justify left)
+		)
+	)
+	(text "Microcontroller"
+		(exclude_from_sim no)
+		(at 33.274 21.844 0)
+		(effects
+			(font
+				(size 2.54 2.54)
+				(thickness 0.508)
+				(bold yes)
+			)
+		)
+	)
 )

Commit message: test
Parts:
- added U1: STM32H7A3IGTxQ, Package_QFP:LQFP-176_24x24mm_P0.5mm, symbol MCU_ST_STM32H7:STM32H7A3IGTxQ
Connections:
- new net: U1.100 (VSS), U1.106 (VSS), U1.112 (VSS), U1.119 (VSS), U1.12 (VSS), U1.134 (VSS), U1.137 (VSS), U1.151 (VSS), U1.159 (VSS), U1.173 (VSS), U1.24 (VSS), U1.45 (VSS), U1.47 (VSS), U1.6 (VSS), U1.64 (VSS), U1.70 (VSS), U1.81 (VSS), U1.83 (VSS), U1.93 (VSS)

Commit message: renew
Parts:
- removed U1: STM32H7A3IGTxQ, Package_QFP:LQFP-176_24x24mm_P0.5mm, symbol MCU_ST_STM32H7:STM32H7A3IGTxQ
