File: NDXPCOMPUTER.kicad_sch (KiCad schematic)
At the start: 0 parts

Commit message: changes
Other:
- note added: "1. git switch master 2. git pull --rebase origin master 3. git checkout -b your-new-branch-name 3. make your changes!! 4. git add . 5. git commit -m "your-descriptive-message" 6. git push origin your-branch-name"
- note removed: "1. git pull --rebase origin master 2. make your changes!! 3. git add . 3. git commit -m "your-descriptive-message" 5. git push origin master"
Changed lines of the file:
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@@
 	(rectangle
 		(start -111.506 56.642)
-		(end -1.016 147.828)
+		(end -1.016 163.83)
 		(stroke
 			(width 0)
@@
 		)
 	)
-	(text "1. git pull --rebase origin master\n2. make your changes!!\n3. git add .\n3. git commit -m \"your-descriptive-message\"\n5. git push origin master"
+	(text "1. git switch master\n2. git pull --rebase origin master\n3. git checkout -b your-new-branch-name\n3. make your changes!!\n4. git add .\n5. git commit -m \"your-descriptive-message\"\n6. git push origin your-branch-name"
 		(exclude_from_sim no)
-		(at -107.188 86.614 0)
+		(at -107.188 92.456 0)
 		(effects
 			(font
@@
 	(text "Do not be afraid to make commits! \nEverything will be reviewed\nand nothing is final! The only way \nto learn is to make mistakes!"
 		(exclude_from_sim no)
-		(at -59.944 133.35 0)
+		(at -60.198 146.05 0)
 		(effects
 			(font
@@
 	(text "Do the above steps each time you sit down to design.\nYou should not start designing without starting at \nthe first step, and should not stop before commiting \nyour changes, whatever they were, to the remote server.\n"
 		(exclude_from_sim no)
-		(at -57.15 106.68 0)
+		(at -57.15 117.094 0)
 		(effects
 			(font
@@
 	(polyline
 		(pts
-			(xy -109.474 118.618) (xy -2.794 118.618)
+			(xy -109.22 129.54) (xy -2.54 129.54)
 		)
 		(stroke

Commit message: renew
Other:
- note added: "1. git switch master 2. git pull --rebase origin master 3. git checkout -b your-new-branch-name 3. make your changes!! 4. git add . 5. git commit -m "your-descriptive-message" 6. git push origin your-branch-name 7. Submit pull request on github"
- note removed: "1. git switch master 2. git pull --rebase origin master 3. git checkout -b your-new-branch-name 3. make your changes!! 4. git add . 5. git commit -m "your-descriptive-message" 6. git push origin your-branch-name"
Changed lines of the file:
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@@
 		)
 	)
-	(text "1. git switch master\n2. git pull --rebase origin master\n3. git checkout -b your-new-branch-name\n3. make your changes!!\n4. git add .\n5. git commit -m \"your-descriptive-message\"\n6. git push origin your-branch-name"
+	(text "1. git switch master\n2. git pull --rebase origin master\n3. git checkout -b your-new-branch-name\n3. make your changes!!\n4. git add .\n5. git commit -m \"your-descriptive-message\"\n6. git push origin your-branch-name\n7. Submit pull request on github"
 		(exclude_from_sim no)
 		(at -107.188 92.456 0)

Commit message: added barometer schematic
Other:
- sheet Barometer ports: added SCLK, SDA; removed none
Changed lines of the file:
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@@
+			)
+		)
+		(pin "SDA" input
+			(at 68.58 115.57 0)
+			(effects
+				(font
+					(size 1.27 1.27)
+				)
+				(justify right)
+			)
+		)
+		(pin "SCLK" input
+			(at 68.58 119.38 0)
+			(effects
+				(font
+					(size 1.27 1.27)
+				)
+				(justify right)
 			)
 		)
